File: latest/Viewer/main-board.kicad_pcb (KiCad board)
At the start: 2 copper layers, 0 parts

Commit message: Update latest build (main@bfcce57)
Other:
- board outline added: 93.5 x 66.5 mm
Changed lines of the file:
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@@
 		)
+	)
+	(gr_rect
+		(start 88.5 49)
+		(end 182 115.5)
+		(stroke
+			(width 0.05)
+			(type default)
+		)
+		(fill no)
+		(layer "Edge.Cuts")
 	)
 	(embedded_fonts no)
