File: latest/Viewer/main-board.kicad_sch (KiCad schematic)
At the start: 0 parts

Commit message: Update latest build (main@bfcce57)
Parts:
- added C1: 1uF, Capacitor_SMD:C_0805_2012Metric_Pad1.18x1.45mm_HandSolder, symbol Device:C
- added C2, C3, C4: 4.7uF, Capacitor_SMD:C_0805_2012Metric_Pad1.18x1.45mm_HandSolder, symbol Device:C
- added J1: USB_C_Receptacle_USB2.0_16P, Package_DFN_QFN:WDFN-10-1EP_3x3mm_P0.5mm_EP1.8x2.5mm, symbol Connector:USB_C_Receptacle_USB2.0_16P
- added Q1: AONR21307, DFN_3X3_EP, symbol Samacsys:AONR21307
- added R1: 10R, Resistor_SMD:R_0805_2012Metric_Pad1.20x1.40mm_HandSolder, symbol Device:R
- added R2: 5K1, Resistor_SMD:R_0805_2012Metric_Pad1.20x1.40mm_HandSolder, symbol Device:R
- added R3: 49K9, Resistor_SMD:R_0805_2012Metric_Pad1.20x1.40mm_HandSolder, symbol Device:R
- added R4, R5: 10R, Resistor_SMD:R_0603_1608Metric_Pad0.98x0.95mm_HandSolder, symbol Device:R
- added U1: HUSB238_xxxDD, Package_DFN_QFN:WDFN-10-1EP_3x3mm_P0.5mm_EP1.8x2.5mm, symbol Interface_USB:HUSB238_xxxDD
Connections:
- new net: R2.1, U1.10 (GATE)
- new net: Q1.4 (G), R2.2, R3.1
- new net: J1.A4 (VBUS), J1.A9 (VBUS), J1.B4 (VBUS), J1.B9 (VBUS), Q1.1 (S_1), Q1.2 (S_2), Q1.3 (S_3), R1.1, R3.2
- new net: J1.A5 (CC1), U1.4 (CC1)
- new net: J1.A6 (D+), J1.B6 (D+), U1.2 (D+)
- new net: J1.A7 (D-), J1.B7 (D-), U1.3 (D-)
- new net: J1.B5 (CC2), U1.5 (CC2)
- new net: C1.2, R1.2, U1.1 (VIN)
- new net: R5.2, U1.9 (ISET)
- new net: R4.1, U1.8 (VSET)
- new net GND: C1.1, C2.2, C3.2, C4.2, J1.A1 (GND), J1.A12 (GND), J1.B1 (GND), J1.B12 (GND), J1.SH (SHIELD), R4.2, R5.1, U1.11 (GND)
- new net PD_SCL: U1.7 (SCL)
- new net PD_SDA: U1.6 (SDA)
- new net VBUS: C2.1, C3.1, C4.1, Q1.5 (D_1), Q1.6 (D_2), Q1.7 (D_3), Q1.8 (D_4)
- no-connect marks 0 -> 2

Commit message: Update latest build (main@2425257)
Parts:
- added C5, C6: 4.7uF, Capacitor_SMD:C_0805_2012Metric_Pad1.18x1.45mm_HandSolder, symbol Device:C
- added C7: 0.1uF, Capacitor_SMD:C_0603_1608Metric_Pad1.08x0.95mm_HandSolder, symbol Device:C
- added C8, C9: 22uF, Capacitor_SMD:C_0603_1608Metric_Pad1.08x0.95mm_HandSolder, symbol Device:C
- added L1: IHLP1616BZER4R7M11, INDPM4441X200N, symbol Samacsys:IHLP1616BZER4R7M11
- added U2: AP63205WU, Package_TO_SOT_SMD:TSOT-23-6_HandSoldering, symbol Regulator_Switching:AP63205WU
- C1: value 1uF -> 4.7uF
Connections:
- net GND: now also C5.2, C6.2, C8.1, C9.1, U2.4 (GND)
- net VBUS: now also C5.1, C6.1, U2.2 (EN), U2.3 (IN)
- new net: C7.2, L1.1, U2.5 (SW)
- new net: C7.1, U2.6 (BST)
- new net +5V: C8.2, C9.2, L1.2, U2.1 (FB)

Commit message: Update latest build (main@d6ce267)
Parts:
- J1: footprint Package_DFN_QFN:WDFN-10-1EP_3x3mm_P0.5mm_EP1.8x2.5mm -> Connector_USB:USB_C_Receptacle_Palconn_UTC16-G
- L1: footprint INDPM4441X200N -> Samacsys:INDPM4441X200N
- Q1: footprint DFN_3X3_EP -> Samacsys:DFN_3X3_EP
Changed lines of the file:
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@@
       (effects (font (size 1.27 1.27)))
     )
-    (property "Footprint" "INDPM4441X200N" (at 125.73 211.76 0) (do_not_autoplace no) (show_name no) (hide yes)
+    (property "Footprint" "Samacsys:INDPM4441X200N" (at 125.73 211.76 0) (do_not_autoplace no) (show_name no) (hide yes)
       (effects (font (size 1.27 1.27)) (justify left top))
     )
@@
       (effects (font (size 1.27 1.27)))
     )
-    (property "Footprint" "Package_DFN_QFN:WDFN-10-1EP_3x3mm_P0.5mm_EP1.8x2.5mm" (at 45.72 58.42 0) (do_not_autoplace no) (show_name no) (hide yes)
+    (property "Footprint" "Connector_USB:USB_C_Receptacle_Palconn_UTC16-G" (at 45.72 58.42 0) (do_not_autoplace no) (show_name no) (hide yes)
       (effects (font (size 1.27 1.27)))
     )
@@
       (effects (font (size 1.27 1.27)))
     )
-    (property "Footprint" "DFN_3X3_EP" (at 133.35 130.48 0) (do_not_autoplace no) (show_name no) (hide yes)
+    (property "Footprint" "Samacsys:DFN_3X3_EP" (at 133.35 130.48 0) (do_not_autoplace no) (show_name no) (hide yes)
       (effects (font (size 1.27 1.27)) (justify left top))
     )

Commit message: Update latest build (main@96a2231)
Parts:
- added C10, C11: 4.7uF, Capacitor_SMD:C_0603_1608Metric_Pad1.08x0.95mm_HandSolder, symbol Device:C
- added U3: AP2112K-3.3, Package_TO_SOT_SMD:SOT-23-5, symbol Regulator_Linear:AP2112K-3.3
Connections:
- net +5V: now also C10.1, U3.1 (VIN), U3.3 (EN)
- net GND: now also C10.2, C11.2, U3.2 (GND)
- new net +3.3V: C11.1, U3.5 (VOUT)

Commit message: Update latest build (main@d69d42a)
Parts:
- added U4: PTR54L, Project_Specific_Parts:PTR54L15, symbol Project_Specific_Parts:PTR54L
Changed lines of the file:
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@@
+    )
+  )
+  (symbol (lib_id "Project_Specific_Parts:PTR54L") (at 196.85 64.77 0) (unit 1) (body_style 1)
+    (exclude_from_sim no) (in_bom yes) (on_board yes) (in_pos_files yes) (dnp no) (fields_autoplaced)
+    (property "Reference" "U4" (at 198.374 53.34 0) (do_not_autoplace no) (show_name no)
+      (effects (font (size 1.27 1.27)))
+    )
+    (property "Value" "PTR54L" (at 200.66 55.626 0) (do_not_autoplace no) (show_name no)
+      (effects (font (size 1.27 1.27)))
+    )
+    (property "Footprint" "Project_Specific_Parts:PTR54L15" (at 196.85 64.77 0) (do_not_autoplace no) (show_name no) (hide yes)
+      (effects (font (size 1.27 1.27)))
+    )
+    (property "Datasheet" "" (at 196.85 64.77 0) (do_not_autoplace no) (show_name no) (hide yes)
+      (effects (font (size 1.27 1.27)))
+    )
+    (property "Description" "" (at 196.85 64.77 0) (do_not_autoplace no) (show_name no) (hide yes)
+      (effects (font (size 1.27 1.27)))
+    )
+    (pin "5")
+    (pin "7")
+    (pin "1")
+    (pin "14")
+    (pin "10")
+    (pin "4")
+    (pin "3")
+    (pin "11")
+    (pin "13")
+    (pin "2")
+    (pin "8")
+    (pin "9")
+    (pin "6")
+    (pin "15")
+    (pin "12")
+    (pin "33")
+    (pin "27")
+    (pin "26")
+    (pin "36")
+    (pin "35")
+    (pin "32")
+    (pin "24")
+    (pin "30")
+    (pin "17")
+    (pin "22")
+    (pin "29")
+    (pin "34")
+    (pin "18")
+    (pin "19")
+    (pin "21")
+    (pin "16")
+    (pin "23")
+    (pin "28")
+    (pin "25")
+    (pin "20")
+    (pin "31")
+    (instances
+      (project "main-board"
+        (path "/fe215afa-a228-4dbb-8560-a0753323a3f2"
+          (reference "U4") (unit 1)
+        )
+      )
     )
   )

Commit message: Update latest build (main@08d4132)
Parts:
- added C12: 100nF, Capacitor_SMD:C_0603_1608Metric_Pad1.08x0.95mm_HandSolder, symbol Device:C
- added C13: 22uF, Capacitor_SMD:C_0603_1608Metric_Pad1.08x0.95mm_HandSolder, symbol Device:C
Connections:
- net +3.3V: now also U4.2 (VCC), C12.2, C13.2
- net GND: now also U4.1 (GND), C12.1, C13.1
Changed lines of the file:
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@@
   (junction (at 43.18 115.57) (diameter 0) (color 0 0 0 0)
   )
+  (junction (at 184.15 52.07) (diameter 0) (color 0 0 0 0)
+  )
   (junction (at 137.16 35.56) (diameter 0) (color 0 0 0 0)
   )
@@
   (junction (at 63.5 60.96) (diameter 0) (color 0 0 0 0)
   )
+  (junction (at 176.53 52.07) (diameter 0) (color 0 0 0 0)
+  )
+  (junction (at 184.15 63.5) (diameter 0) (color 0 0 0 0)
+  )
   (junction (at 54.61 123.19) (diameter 0) (color 0 0 0 0)
   )
   (junction (at 137.16 38.1) (diameter 0) (color 0 0 0 0)
+  )
+  (junction (at 176.53 63.5) (diameter 0) (color 0 0 0 0)
   )
   (junction (at 52.07 166.37) (diameter 0) (color 0 0 0 0)
@@
     (stroke (width 0) (type default))
   )
+  (wire (pts (xy 176.53 63.5) (xy 176.53 69.85))
+    (stroke (width 0) (type default))
+  )
   (wire (pts (xy 57.15 55.88) (xy 60.96 55.88))
     (stroke (width 0) (type default))
@@
     (stroke (width 0) (type default))
   )
+  (wire (pts (xy 176.53 52.07) (xy 176.53 63.5))
+    (stroke (width 0) (type default))
+  )
   (wire (pts (xy 88.9 48.26) (xy 90.17 48.26))
     (stroke (width 0) (type default))
@@
     (stroke (width 0) (type default))
   )
+  (wire (pts (xy 194.31 67.31) (xy 184.15 67.31))
+    (stroke (width 0) (type default))
+  )
   (wire (pts (xy 93.98 27.94) (xy 107.95 27.94))
     (stroke (width 0) (type default))
@@
     (stroke (width 0) (type default))
   )
+  (wire (pts (xy 194.31 69.85) (xy 176.53 69.85))
+    (stroke (width 0) (type default))
+  )
   (wire (pts (xy 102.87 69.85) (xy 102.87 71.12))
     (stroke (width 0) (type default))
@@
     (stroke (width 0) (type default))
   )
+  (wire (pts (xy 184.15 63.5) (xy 184.15 67.31))
+    (stroke (width 0) (type default))
+  )
   (wire (pts (xy 35.56 115.57) (xy 43.18 115.57))
     (stroke (width 0) (type default))
@@
   )
   (wire (pts (xy 137.16 27.94) (xy 137.16 35.56))
+    (stroke (width 0) (type default))
+  )
+  (wire (pts (xy 184.15 52.07) (xy 184.15 63.5))
     (stroke (width 0) (type default))
   )
@@
         (path "/fe215afa-a228-4dbb-8560-a0753323a3f2"
           (reference "#PWR012") (unit 1)
+        )
+      )
+    )
+  )
+  (symbol (lib_id "power:GND") (at 184.15 52.07 90) (unit 1) (body_style 1)
+    (exclude_from_sim no) (in_bom yes) (on_board yes) (in_pos_files yes) (dnp no) (fields_autoplaced)
+    (property "Reference" "#PWR016" (at 190.5 52.07 0) (do_not_autoplace no) (show_name no) (hide yes)
+      (effects (font (size 1.27 1.27)))
+    )
+    (property "Value" "GND" (at 187.96 52.0699 90) (do_not_autoplace no) (show_name no)
+      (effects (font (size 1.27 1.27)) (justify right))
+    )
+    (property "Footprint" "" (at 184.15 52.07 0) (do_not_autoplace no) (show_name no) (hide yes)
+      (effects (font (size 1.27 1.27)))
+    )
+    (property "Datasheet" "" (at 184.15 52.07 0) (do_not_autoplace no) (show_name no) (hide yes)
+      (effects (font (size 1.27 1.27)))
+    )
+    (property "Description" "Power symbol creates a global label with name \"GND\" , ground" (at 184.15 52.07 0) (do_not_autoplace no) (show_name no) (hide yes)
+      (effects (font (size 1.27 1.27)))
+    )
+    (pin "1")
+    (instances
+      (project "main-board"
+        (path "/fe215afa-a228-4dbb-8560-a0753323a3f2"
+          (reference "#PWR016") (unit 1)
         )
       )
@@
     )
   )
+  (symbol (lib_id "Device:C") (at 180.34 63.5 270) (unit 1) (body_style 1)
+    (exclude_from_sim no) (in_bom yes) (on_board yes) (in_pos_files yes) (dnp no) (fields_autoplaced)
+    (property "Reference" "C12" (at 180.34 55.88 90) (do_not_autoplace no) (show_name no)
+      (effects (font (size 1.27 1.27)))
+    )
+    (property "Value" "100nF" (at 180.34 58.42 90) (do_not_autoplace no) (show_name no)
+      (effects (font (size 1.27 1.27)))
+    )
+    (property "Footprint" "Capacitor_SMD:C_0603_1608Metric_Pad1.08x0.95mm_HandSolder" (at 176.53 64.4652 0) (do_not_autoplace no) (show_name no) (hide yes)
+      (effects (font (size 1.27 1.27)))
+    )
+    (property "Datasheet" "" (at 180.34 63.5 0) (do_not_autoplace no) (show_name no) (hide yes)
+      (effects (font (size 1.27 1.27)))
+    )
+    (property "Description" "Unpolarized capacitor" (at 180.34 63.5 0) (do_not_autoplace no) (show_name no) (hide yes)
+      (effects (font (size 1.27 1.27)))
+    )
+    (pin "2")
+    (pin "1")
+    (instances
+      (project "main-board"
+        (path "/fe215afa-a228-4dbb-8560-a0753323a3f2"
+          (reference "C12") (unit 1)
+        )
+      )
+    )
+  )
   (symbol (lib_id "Device:C") (at 170.18 34.29 0) (unit 1) (body_style 1)
     (exclude_from_sim no) (in_bom yes) (on_board yes) (in_pos_files yes) (dnp no) (fields_autoplaced)
@@
     )
   )
+  (symbol (lib_id "power:+3.3V") (at 176.53 52.07 90) (unit 1) (body_style 1)
+    (exclude_from_sim no) (in_bom yes) (on_board yes) (in_pos_files yes) (dnp no) (fields_autoplaced)
+    (property "Reference" "#PWR015" (at 180.34 52.07 0) (do_not_autoplace no) (show_name no) (hide yes)
+      (effects (font (size 1.27 1.27)))
+    )
+    (property "Value" "+3.3V" (at 172.72 52.0699 90) (do_not_autoplace no) (show_name no)
+      (effects (font (size 1.27 1.27)) (justify left))
+    )
+    (property "Footprint" "" (at 176.53 52.07 0) (do_not_autoplace no) (show_name no) (hide yes)
+      (effects (font (size 1.27 1.27)))
+    )
+    (property "Datasheet" "" (at 176.53 52.07 0) (do_not_autoplace no) (show_name no) (hide yes)
+      (effects (font (size 1.27 1.27)))
+    )
+    (property "Description" "Power symbol creates a global label with name \"+3.3V\"" (at 176.53 52.07 0) (do_not_autoplace no) (show_name no) (hide yes)
+      (effects (font (size 1.27 1.27)))
+    )
+    (pin "1")
+    (instances
+      (project "main-board"
+        (path "/fe215afa-a228-4dbb-8560-a0753323a3f2"
+          (reference "#PWR015") (unit 1)
+        )
+      )
+    )
+  )
   (symbol (lib_id "power:GND") (at 144.78 127 0) (unit 1) (body_style 1)
     (exclude_from_sim no) (in_bom yes) (on_board yes) (in_pos_files yes) (dnp no) (fields_autoplaced)
@@
         )
       )
+    )
+  )
+  (symbol (lib_id "Device:C") (at 180.34 52.07 270) (unit 1) (body_style 1)
+    (exclude_from_sim no) (in_bom yes) (on_board yes) (in_pos_files yes) (dnp no) (fields_autoplaced)
+    (property "Reference" "C13" (at 180.34 44.45 90) (do_not_autoplace no) (show_name no)
+      (effects (font (size 1.27 1.27)))
+    )
+    (property "Value" "22uF" (at 180.34 46.99 90) (do_not_autoplace no) (show_name no)
+      (effects (font (size 1.27 1.27)))
+    )
+    (property "Footprint" "Capacitor_SMD:C_0603_1608Metric_Pad1.08x0.95mm_HandSolder" (at 176.53 53.0352 0) (do_not_autoplace no) (show_name no) (hide yes)
+      (effects (font (size 1.27 1.27)))
+    )
+    (property "Datasheet" "" (at 180.34 52.07 0) (do_not_autoplace no) (show_name no) (hide yes)
+      (effects (font (size 1.27 1.27)))
+    )
+    (property "Description" "Unpolarized capacitor" (at 180.34 52.07 0) (do_not_autoplace no) (show_name no) (hide yes)
+      (effects (font (size 1.27 1.27)))
+    )
+    (pin "2")
+    (pin "1")
+    (instances
+      (project "main-board"
+        (path "/fe215afa-a228-4dbb-8560-a0753323a3f2"
+          (reference "C13") (unit 1)
+        )
+      )

Commit message: Update latest build (main@0e79090)
Parts:
- added U5: TMC2226-SA, Package_SO:HTSSOP-28-1EP_4.4x9.7mm_P0.65mm_EP2.75x6.2mm_ThermalVias, symbol Driver_Motor:TMC2226-SA
- C12: value 100nF -> 0.1uF
Connections:
- new net: U5.22 (GND), U5.29 (GND), U5.6 (GND)
Other:
- moved on the sheet: C1, C10, C11, C12, C13, C2, C3, C4, C5, C6, C7, C8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

Commit message: Update latest build (main@a210432)
Parts:
- U2: footprint Package_TO_SOT_SMD:TSOT-23-6_HandSoldering -> Package_TO_SOT_SMD:TSOT-23-6
Changed lines of the file:
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@@
       (effects (font (size 1.27 1.27)))
     )
-    (property "Footprint" "Package_TO_SOT_SMD:TSOT-23-6_HandSoldering" (at 97.79 179.07 0) (do_not_autoplace no) (show_name no) (hide yes)
+    (property "Footprint" "Package_TO_SOT_SMD:TSOT-23-6" (at 97.79 179.07 0) (do_not_autoplace no) (show_name no) (hide yes)
       (effects (font (size 1.27 1.27)))
     )
