File: latest/Viewer/main-board.kicad_sch (KiCad schematic)
At the start: 66 parts, among them J1 USB_C_Receptacle_USB2.0_16P, J2 S4B-XH-A_LF__SN_, J3 S4B-XH-A_LF__SN_, J4 Conn_ARM_JTAG_SWD_10, Q1 AONR21307, U1 HUSB238_xxxDD, U2 AP63205WU, U3 AP2112K-3.3, U4 PTR54L, U5 TMC2226-SA, U6 TMC2226-SA

Commit message: Update latest build (main@dce9144)
Parts:
- removed R16, R17: 82R, Resistor_SMD:R_0603_1608Metric_Pad0.98x0.95mm_HandSolder, symbol Device:R
- removed R18: 300R, Resistor_SMD:R_0603_1608Metric_Pad0.98x0.95mm_HandSolder, symbol Device:R
- added U7: KTD2026BEWE-TR, Project_Specific_Parts:UTDFN8_1P5X1P5_KIN, symbol Project_Specific_Parts:KTD2026BEWE-TR
Connections:
- net +3.3V: now also U7.5 (VIN)
- net BLUE: now also LED1.4, U7.2 (D3)
- net GND: now also U7.8 (GND), U7.9 (GND)
- net GREEN: now also LED1.2, U7.3 (D2)
- net RED: now also LED1.3, U7.4 (D1)
- new net SCL_KTD: U7.6 (SCL)
- new net SDA_KTD: U7.7 (SDA)
- new net STATUS_KTD: U7.1 (ST)
Other:
- moved on the sheet: LED1

Commit message: Update latest build (main@6556eb7)
Parts:
- added C36: 4.7uF, Capacitor_SMD:C_0805_2012Metric_Pad1.18x1.45mm_HandSolder, symbol Device:C
Connections:
- net +3.3V: now also C36.1
- net GND: now also C36.2
Changed lines of the file:
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@@
   (junction (at 233.68 41.91) (diameter 0) (color 0 0 0 0)
   )
+  (junction (at 133.35 119.38) (diameter 0) (color 0 0 0 0)
+  )
   (junction (at 135.89 44.45) (diameter 0) (color 0 0 0 0)
   )
@@
     )
   )
+  (symbol (lib_id "Device:C") (at 133.35 123.19 0) (unit 1) (body_style 1)
+    (exclude_from_sim no) (in_bom yes) (on_board yes) (in_pos_files yes) (dnp no) (fields_autoplaced)
+    (property "Reference" "C36" (at 137.16 121.9199 0) (do_not_autoplace no) (show_name no)
+      (effects (font (size 1.27 1.27)) (justify left))
+    )
+    (property "Value" "4.7uF" (at 137.16 124.4599 0) (do_not_autoplace no) (show_name no)
+      (effects (font (size 1.27 1.27)) (justify left))
+    )
+    (property "Footprint" "Capacitor_SMD:C_0805_2012Metric_Pad1.18x1.45mm_HandSolder" (at 134.3152 127 0) (do_not_autoplace no) (show_name no) (hide yes)
+      (effects (font (size 1.27 1.27)))
+    )
+    (property "Datasheet" "" (at 133.35 123.19 0) (do_not_autoplace no) (show_name no) (hide yes)
+      (effects (font (size 1.27 1.27)))
+    )
+    (property "Description" "Unpolarized capacitor X7R" (at 133.35 123.19 0) (do_not_autoplace no) (show_name no) (hide yes)
+      (effects (font (size 1.27 1.27)))
+    )
+    (pin "2")
+    (pin "1")
+    (instances
+      (project "main-board"
+        (path "/fe215afa-a228-4dbb-8560-a0753323a3f2"
+          (reference "C36") (unit 1)
+        )
+      )
+    )
+  )
   (symbol (lib_id "power:+3.3V") (at 368.3 77.47 180) (unit 1) (body_style 1)
     (exclude_from_sim no) (in_bom yes) (on_board yes) (in_pos_files yes) (dnp no) (fields_autoplaced)
@@
         )
       )
+    )
+  )
+  (symbol (lib_id "power:GND") (at 133.35 127 0) (unit 1) (body_style 1)
+    (exclude_from_sim no) (in_bom yes) (on_board yes) (in_pos_files yes) (dnp no) (fields_autoplaced)
+    (property "Reference" "#PWR054" (at 133.35 133.35 0) (do_not_autoplace no) (show_name no) (hide yes)
+      (effects (font (size 1.27 1.27)))
+    )
+    (property "Value" "GND" (at 133.35 132.08 0) (do_not_autoplace no) (show_name no)
+      (effects (font (size 1.27 1.27)))
+    )
+    (property "Footprint" "" (at 133.35 127 0) (do_not_autoplace no) (show_name no) (hide yes)
+      (effects (font (size 1.27 1.27)))
+    )
+    (property "Datasheet" "" (at 133.35 127 0) (do_not_autoplace no) (show_name no) (hide yes)
+      (effects (font (size 1.27 1.27)))
+    )
+    (property "Description" "Power symbol creates a global label with name \"GND\" , ground" (at 133.35 127 0) (do_not_autoplace no) (show_name no) (hide yes)
+      (effects (font (size 1.27 1.27)))
+    )
+    (pin "1")
+    (instances
+      (project "main-board"
+        (path "/fe215afa-a228-4dbb-8560-a0753323a3f2"
+          (reference "#PWR054") (unit 1)
+        )
+      )

Commit message: Update latest build (main@d184ee7)
Connections:
- net DIAG1: no longer U6.15 (DIAG)
- net DIR1: no longer U6.23 (DIR)
- net EN1: no longer R14.2, U6.5 (~{EN})
- net STEP1: no longer U6.20 (STEP)
- net UART_RX renamed UART_RX1
- net UART_RX1: no longer R11.1, U6.18 (PDN_UART)
- net UART_TX renamed UART_TX1
- net UART_TX1: no longer R11.2
- net VREF renamed VREF1
- net VREF1: no longer C24.2, R15.1, U6.11 (5VOUT)
- new net DIAG2: U6.15 (DIAG)
- new net DIR2: U6.23 (DIR)
- new net EN2: R14.2, U6.5 (~{EN})
- new net STEP2: U6.20 (STEP)
- new net UART_RX2: R11.1, U6.18 (PDN_UART)
- new net UART_TX2: R11.2
- new net VREF2: C24.2, R15.1, U6.11 (5VOUT)
Changed lines of the file:
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@@
     (effects (font (size 1.27 1.27)) (justify right bottom))
   )
-  (label "VREF" (at 210.82 160.02 0)
+  (label "VREF1" (at 210.82 160.02 0)
     (effects (font (size 1.27 1.27)) (justify left bottom))
   )
@@
     (effects (font (size 1.27 1.27)) (justify left bottom))
   )
-  (label "UART_RX" (at 184.15 185.42 0)
+  (label "UART_RX1" (at 184.15 185.42 0)
     (effects (font (size 1.27 1.27)) (justify left bottom))
   )
@@
     (effects (font (size 1.27 1.27)) (justify left bottom))
   )
-  (label "VREF" (at 299.72 218.44 180)
-    (effects (font (size 1.27 1.27)) (justify right bottom))
-  )
-  (label "UART_TX" (at 171.45 182.88 180)
+  (label "VREF2" (at 299.72 218.44 180)
+    (effects (font (size 1.27 1.27)) (justify right bottom))
+  )
+  (label "UART_TX1" (at 171.45 182.88 180)
     (effects (font (size 1.27 1.27)) (justify right bottom))
   )
@@
     (effects (font (size 1.27 1.27)) (justify left bottom))
   )
-  (label "DIAG1" (at 307.34 210.82 0)
+  (label "DIAG2" (at 307.34 210.82 0)
     (effects (font (size 1.27 1.27)) (justify left bottom))
   )
@@
     (effects (font (size 1.27 1.27)) (justify right bottom))
   )
-  (label "DIR1" (at 307.34 190.5 0)
-    (effects (font (size 1.27 1.27)) (justify left bottom))
-  )
-  (label "VREF" (at 328.93 160.02 0)
+  (label "DIR2" (at 307.34 190.5 0)
+    (effects (font (size 1.27 1.27)) (justify left bottom))
+  )
+  (label "VREF2" (at 328.93 160.02 0)
     (effects (font (size 1.27 1.27)) (justify left bottom))
   )
@@
     (effects (font (size 1.27 1.27)) (justify left bottom))
   )
-  (label "UART_TX" (at 289.56 182.88 180)
-    (effects (font (size 1.27 1.27)) (justify right bottom))
-  )
-  (label "VREF" (at 181.61 218.44 180)
+  (label "UART_TX2" (at 289.56 182.88 180)
+    (effects (font (size 1.27 1.27)) (justify right bottom))
+  )
+  (label "VREF1" (at 181.61 218.44 180)
     (effects (font (size 1.27 1.27)) (justify right bottom))
   )
@@
     (effects (font (size 1.27 1.27)) (justify right bottom))
   )
-  (label "STEP1" (at 307.34 187.96 0)
+  (label "STEP2" (at 307.34 187.96 0)
     (effects (font (size 1.27 1.27)) (justify left bottom))
   )
@@
     (effects (font (size 1.27 1.27)) (justify left bottom))
   )
-  (label "UART_RX" (at 302.26 185.42 0)
+  (label "UART_RX2" (at 302.26 185.42 0)
     (effects (font (size 1.27 1.27)) (justify left bottom))
   )
@@
     (effects (font (size 1.27 1.27)) (justify left bottom))
   )
-  (label "EN1" (at 307.34 203.2 0)
+  (label "EN2" (at 307.34 203.2 0)
     (effects (font (size 1.27 1.27)) (justify left bottom))
   )
@@
   )
   (symbol (lib_id "Project_Specific_Parts:KTD2026BEWE-TR") (at 92.71 109.22 0) (unit 1) (body_style 1)
-    (exclude_from_sim no) (in_bom yes) (on_board yes) (in_pos_files yes) (dnp no) (fields_autoplaced)
-    (property "Reference" "U7" (at 113.03 99.06 0) (do_not_autoplace no) (show_name no)
+    (exclude_from_sim no) (in_bom yes) (on_board yes) (in_pos_files yes) (dnp no)
+    (property "Reference" "U7" (at 104.394 99.568 0) (do_not_autoplace no) (show_name no)
       (effects (font (size 1.524 1.524)))
     )

Commit message: Update latest build (main@8744ec9)
Parts:
- removed R8: 1K, Resistor_SMD:R_0603_1608Metric_Pad0.98x0.95mm_HandSolder, symbol Device:R
Connections:
- net UART_RX2 is gone; now on net UART_RX: R11.1, U6.18 (PDN_UART)
- net UART_RX1 renamed UART_RX
- net UART_TX2 renamed UART_TX
Other:
- moved on the sheet: R11
Changed lines of the file:
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@@
   (junction (at 125.73 152.4) (diameter 0) (color 0 0 0 0)
   )
-  (junction (at 302.26 182.88) (diameter 0) (color 0 0 0 0)
-  )
   (junction (at 104.14 152.4) (diameter 0) (color 0 0 0 0)
   )
@@
   (junction (at 368.3 187.96) (diameter 0) (color 0 0 0 0)
   )
-  (junction (at 184.15 182.88) (diameter 0) (color 0 0 0 0)
-  )
   (junction (at 63.5 232.41) (diameter 0) (color 0 0 0 0)
   )
@@
     (stroke (width 0) (type default))
   )
-  (wire (pts (xy 298.45 182.88) (xy 302.26 182.88))
-    (stroke (width 0) (type default))
-  )
   (wire (pts (xy 104.14 152.4) (xy 105.41 152.4))
     (stroke (width 0) (type default))
@@
     (stroke (width 0) (type default))
   )
-  (wire (pts (xy 289.56 182.88) (xy 290.83 182.88))
-    (stroke (width 0) (type default))
-  )
   (wire (pts (xy 102.87 52.07) (xy 106.68 52.07))
     (stroke (width 0) (type default))
@@
     (stroke (width 0) (type default))
   )
+  (wire (pts (xy 257.81 228.6) (xy 266.7 228.6))
+    (stroke (width 0) (type default))
+  )
   (wire (pts (xy 368.3 187.96) (xy 368.3 189.23))
     (stroke (width 0) (type default))
@@
     (stroke (width 0) (type default))
   )
-  (wire (pts (xy 184.15 182.88) (xy 184.15 185.42))
+  (wire (pts (xy 311.15 149.86) (xy 311.15 157.48))
     (stroke (width 0) (type default))
   )
-  (wire (pts (xy 311.15 149.86) (xy 311.15 157.48))
+  (wire (pts (xy 274.32 228.6) (xy 283.21 228.6))
     (stroke (width 0) (type default))
   )
@@
     (stroke (width 0) (type default))
   )
-  (wire (pts (xy 184.15 182.88) (xy 198.12 182.88))
+  (wire (pts (xy 189.23 182.88) (xy 198.12 182.88))
     (stroke (width 0) (type default))
   )
@@
     (stroke (width 0) (type default))
   )
-  (wire (pts (xy 180.34 182.88) (xy 184.15 182.88))
-    (stroke (width 0) (type default))
-  )
   (wire (pts (xy 55.88 57.15) (xy 67.31 57.15))
     (stroke (width 0) (type default))
@@
     (stroke (width 0) (type default))
   )
-  (wire (pts (xy 302.26 182.88) (xy 316.23 182.88))
+  (wire (pts (xy 307.34 182.88) (xy 316.23 182.88))
     (stroke (width 0) (type default))
   )
@@
     (stroke (width 0) (type default))
   )
-  (wire (pts (xy 302.26 182.88) (xy 302.26 185.42))
-    (stroke (width 0) (type default))
-  )
   (wire (pts (xy 233.68 53.34) (xy 233.68 57.15))
     (stroke (width 0) (type default))
@@
     (stroke (width 0) (type default))
   )
-  (wire (pts (xy 171.45 182.88) (xy 172.72 182.88))
-    (stroke (width 0) (type default))
-  )
   (wire (pts (xy 228.6 185.42) (xy 232.41 185.42))
     (stroke (width 0) (type default))
@@
     (effects (font (size 1.27 1.27)) (justify left bottom))
   )
-  (label "UART_RX1" (at 184.15 185.42 0)
+  (label "UART_RX" (at 189.23 182.88 0)
     (effects (font (size 1.27 1.27)) (justify left bottom))
   )
@@
     (effects (font (size 1.27 1.27)) (justify right bottom))
   )
-  (label "UART_TX1" (at 171.45 182.88 180)
-    (effects (font (size 1.27 1.27)) (justify right bottom))
-  )
   (label "SWDIO" (at 347.98 62.23 0)
     (effects (font (size 1.27 1.27)) (justify left bottom))
@@
     (effects (font (size 1.27 1.27)) (justify left bottom))
   )
-  (label "UART_TX2" (at 289.56 182.88 180)
+  (label "UART_RX" (at 283.21 228.6 180)
     (effects (font (size 1.27 1.27)) (justify right bottom))
   )
@@
     (effects (font (size 1.27 1.27)) (justify right bottom))
   )
+  (label "UART_TX" (at 257.81 228.6 0)
+    (effects (font (size 1.27 1.27)) (justify left bottom))
+  )
   (label "GREEN" (at 195.58 119.38 180)
     (effects (font (size 1.27 1.27)) (justify right bottom))
@@
     (effects (font (size 1.27 1.27)) (justify left bottom))
   )
-  (label "UART_RX2" (at 302.26 185.42 0)
+  (label "UART_RX" (at 307.34 182.88 0)
     (effects (font (size 1.27 1.27)) (justify left bottom))
   )
@@
     )
   )
-  (symbol (lib_id "Device:R") (at 176.53 182.88 270) (mirror x) (unit 1) (body_style 1)
-    (exclude_from_sim no) (in_bom yes) (on_board yes) (in_pos_files yes) (dnp no)
-    (property "Reference" "R8" (at 176.53 187.706 90) (do_not_autoplace no) (show_name no)
-      (effects (font (size 1.27 1.27)))
-    )
-    (property "Value" "1K" (at 176.53 185.166 90) (do_not_autoplace no) (show_name no)
-      (effects (font (size 1.27 1.27)))
-    )
-    (property "Footprint" "Resistor_SMD:R_0603_1608Metric_Pad0.98x0.95mm_HandSolder" (at 176.53 184.658 90) (do_not_autoplace no) (show_name no) (hide yes)
-      (effects (font (size 1.27 1.27)))
-    )
-    (property "Datasheet" "" (at 176.53 182.88 0) (do_not_autoplace no) (show_name no) (hide yes)
-      (effects (font (size 1.27 1.27)))
-    )
-    (property "Description" "Resistor" (at 176.53 182.88 0) (do_not_autoplace no) (show_name no) (hide yes)
-      (effects (font (size 1.27 1.27)))
-    )
-    (pin "1")
-    (pin "2")
-    (instances
-      (project "main-board"
-        (path "/fe215afa-a228-4dbb-8560-a0753323a3f2"
-          (reference "R8") (unit 1)
-        )
-      )
-    )
-  )
   (symbol (lib_id "Regulator_Switching:AP63205WU") (at 78.74 154.94 0) (unit 1) (body_style 1)
     (exclude_from_sim no) (in_bom yes) (on_board yes) (in_pos_files yes) (dnp no) (fields_autoplaced)
@@
     )
   )
-  (symbol (lib_id "Device:R") (at 294.64 182.88 270) (mirror x) (unit 1) (body_style 1)
+  (symbol (lib_id "Device:R") (at 270.51 228.6 270) (mirror x) (unit 1) (body_style 1)
     (exclude_from_sim no) (in_bom yes) (on_board yes) (in_pos_files yes) (dnp no)
-    (property "Reference" "R11" (at 294.64 187.706 90) (do_not_autoplace no) (show_name no)
+    (property "Reference" "R11" (at 270.51 233.426 90) (do_not_autoplace no) (show_name no)
       (effects (font (size 1.27 1.27)))
     )
-    (property "Value" "1K" (at 294.64 185.166 90) (do_not_autoplace no) (show_name no)
+    (property "Value" "1K" (at 270.51 230.886 90) (do_not_autoplace no) (show_name no)
       (effects (font (size 1.27 1.27)))
     )
-    (property "Footprint" "Resistor_SMD:R_0603_1608Metric_Pad0.98x0.95mm_HandSolder" (at 294.64 184.658 90) (do_not_autoplace no) (show_name no) (hide yes)
+    (property "Footprint" "Resistor_SMD:R_0603_1608Metric_Pad0.98x0.95mm_HandSolder" (at 270.51 230.378 90) (do_not_autoplace no) (show_name no) (hide yes)
       (effects (font (size 1.27 1.27)))
     )
-    (property "Datasheet" "" (at 294.64 182.88 0) (do_not_autoplace no) (show_name no) (hide yes)
+    (property "Datasheet" "" (at 270.51 228.6 0) (do_not_autoplace no) (show_name no) (hide yes)
       (effects (font (size 1.27 1.27)))
     )
-    (property "Description" "Resistor" (at 294.64 182.88 0) (do_not_autoplace no) (show_name no) (hide yes)
+    (property "Description" "Resistor" (at 270.51 228.6 0) (do_not_autoplace no) (show_name no) (hide yes)
       (effects (font (size 1.27 1.27)))
     )

Commit message: Update latest build (main@b6da3ae)
Parts:
- added R16, R17: 2K2, Resistor_SMD:R_0603_1608Metric_Pad0.98x0.95mm_HandSolder, symbol Device:R
Connections:
- net SCL_KTD is gone; now on net PD_SCL: U7.6 (SCL)
- net SDA_KTD is gone; now on net PD_SDA: U7.7 (SDA)
- net UART_TX is gone; now on an unnamed net: R11.2
- net +3.3V: now also R16.2, R17.2
- net DIAG1: now also U4.29 (P0.00)
- net DIAG2: now also U4.30 (P0.01)
- net PD_SCL: now also U4.33 (P0.04), R17.1
- net PD_SDA: now also U4.32 (P0.03), R16.1
- net UART_RX: now also U4.25 (P2.07)
Other:
- moved on the sheet: R11

Commit message: Update latest build (main@c2d3f34)
Connections:
- net DIAG1: now also U4.8 (P1.14); no longer U4.29 (P0.00)
- net DIAG2: now also U4.17 (P1.08); no longer U4.30 (P0.01)
- net DIR1: now also U4.14 (P1.05)
- net DIR2: now also U4.18 (P2.03)
- net EN1: now also U4.15 (P1.06)
- net EN2: now also U4.19 (P2.04)
- net STEP1: now also U4.13 (P1.04)
- net STEP2: now also U4.16 (P1.07)
- net SWO: now reaches U4.23 (P2.02)
- net SWO: now also J4.6 (SWO/TDO)
- net STATUS_KTD: no longer names the net of U7.1 (ST)
- no-connect marks 12 -> 16
Changed lines of the file:
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@@
   (junction (at 232.41 180.34) (diameter 0) (color 0 0 0 0)
   )
+  (no_connect (at 92.71 109.22))
+  (no_connect (at 243.84 78.74))
   (no_connect (at 355.6 57.15))
   (no_connect (at 198.12 223.52))
   (no_connect (at 316.23 213.36))
   (no_connect (at 198.12 213.36))
+  (no_connect (at 243.84 83.82))
   (no_connect (at 55.88 80.01))
   (no_connect (at 198.12 205.74))
   (no_connect (at 334.01 231.14))
+  (no_connect (at 243.84 86.36))
   (no_connect (at 215.9 231.14))
   (no_connect (at 316.23 223.52))
   (no_connect (at 316.23 205.74))
   (no_connect (at 55.88 82.55))
-  (no_connect (at 355.6 59.69))
+  (no_connect (at 243.84 81.28))
   (wire (pts (xy 189.23 172.72) (xy 189.23 170.18))
     (stroke (width 0) (type default))
@@
     (stroke (width 0) (type default))
   )
+  (wire (pts (xy 259.08 101.6) (xy 259.08 111.76))
+    (stroke (width 0) (type default))
+  )
+  (wire (pts (xy 233.68 88.9) (xy 243.84 88.9))
+    (stroke (width 0) (type default))
+  )
   (wire (pts (xy 88.9 152.4) (xy 104.14 152.4))
     (stroke (width 0) (type default))
@@
     (stroke (width 0) (type default))
   )
+  (wire (pts (xy 276.86 101.6) (xy 276.86 111.76))
+    (stroke (width 0) (type default))
+  )
   (wire (pts (xy 347.98 214.63) (xy 349.25 214.63))
     (stroke (width 0) (type default))
@@
     (stroke (width 0) (type default))
   )
+  (wire (pts (xy 256.54 101.6) (xy 256.54 111.76))
+    (stroke (width 0) (type default))
+  )
   (wire (pts (xy 96.52 232.41) (xy 110.49 232.41))
     (stroke (width 0) (type default))
@@
     (stroke (width 0) (type default))
   )
+  (wire (pts (xy 254 101.6) (xy 254 111.76))
+    (stroke (width 0) (type default))
+  )
   (wire (pts (xy 194.31 167.64) (xy 171.45 167.64))
     (stroke (width 0) (type default))
@@
     (stroke (width 0) (type default))
   )
+  (wire (pts (xy 233.68 76.2) (xy 243.84 76.2))
+    (stroke (width 0) (type default))
+  )
   (wire (pts (xy 81.28 116.84) (xy 92.71 116.84))
     (stroke (width 0) (type default))
@@
     (stroke (width 0) (type default))
   )
-  (wire (pts (xy 81.28 109.22) (xy 92.71 109.22))
-    (stroke (width 0) (type default))
-  )
   (wire (pts (xy 307.34 175.26) (xy 307.34 177.8))
     (stroke (width 0) (type default))
@@
     (stroke (width 0) (type default))
   )
-  (wire (pts (xy 287.02 76.2) (xy 306.07 76.2))
-    (stroke (width 0) (type default))
-  )
   (wire (pts (xy 326.39 157.48) (xy 326.39 165.1))
     (stroke (width 0) (type default))
@@
     (stroke (width 0) (type default))
   )
+  (wire (pts (xy 261.62 101.6) (xy 261.62 111.76))
+    (stroke (width 0) (type default))
+  )
   (wire (pts (xy 77.47 232.41) (xy 77.47 234.95))
     (stroke (width 0) (type default))
@@
     (stroke (width 0) (type default))
   )
+  (wire (pts (xy 266.7 101.6) (xy 266.7 111.76))
+    (stroke (width 0) (type default))
+  )
   (wire (pts (xy 307.34 182.88) (xy 316.23 182.88))
     (stroke (width 0) (type default))
@@
     (stroke (width 0) (type default))
   )
+  (wire (pts (xy 264.16 101.6) (xy 264.16 111.76))
+    (stroke (width 0) (type default))
+  )
   (wire (pts (xy 287.02 59.69) (xy 293.37 59.69))
     (stroke (width 0) (type default))
@@
     (stroke (width 0) (type default))
   )
+  (wire (pts (xy 347.98 59.69) (xy 355.6 59.69))
+    (stroke (width 0) (type default))
+  )
   (wire (pts (xy 110.49 240.03) (xy 110.49 242.57))
     (stroke (width 0) (type default))
@@
     (stroke (width 0) (type default))
   )
-  (wire (pts (xy 287.02 73.66) (xy 306.07 73.66))
-    (stroke (width 0) (type default))
-  )
   (wire (pts (xy 77.47 72.39) (xy 77.47 74.93))
     (stroke (width 0) (type default))
@@
     (effects (font (size 1.27 1.27)) (justify left bottom))
   )
+  (label "SWO" (at 347.98 59.69 0)
+    (effects (font (size 1.27 1.27)) (justify left bottom))
+  )
   (label "SWDIO" (at 293.37 59.69 180)
     (effects (font (size 1.27 1.27)) (justify right bottom))
@@
     (effects (font (size 1.27 1.27)) (justify left bottom))
   )
+  (label "STEP2" (at 259.08 111.76 90)
+    (effects (font (size 1.27 1.27)) (justify left bottom))
+  )
+  (label "DIR1" (at 254 111.76 90)
+    (effects (font (size 1.27 1.27)) (justify left bottom))
+  )
   (label "UART_RX" (at 189.23 182.88 0)
     (effects (font (size 1.27 1.27)) (justify left bottom))
   )
+  (label "EN1" (at 256.54 111.76 90)
+    (effects (font (size 1.27 1.27)) (justify left bottom))
+  )
   (label "GREEN" (at 81.28 114.3 0)
     (effects (font (size 1.27 1.27)) (justify left bottom))
@@
     (effects (font (size 1.27 1.27)) (justify right bottom))
   )
+  (label "STEP1" (at 233.68 88.9 0)
+    (effects (font (size 1.27 1.27)) (justify left bottom))
+  )
   (label "SWDIO" (at 347.98 62.23 0)
     (effects (font (size 1.27 1.27)) (justify left bottom))
@@
     (effects (font (size 1.27 1.27)) (justify right bottom))
   )
+  (label "EN2" (at 266.7 111.76 90)
+    (effects (font (size 1.27 1.27)) (justify left bottom))
+  )
   (label "DIR2" (at 307.34 190.5 0)
     (effects (font (size 1.27 1.27)) (justify left bottom))
@@
     (effects (font (size 1.27 1.27)) (justify right bottom))
   )
+  (label "DIR2" (at 264.16 111.76 90)
+    (effects (font (size 1.27 1.27)) (justify left bottom))
+  )
   (label "GREEN" (at 195.58 119.38 180)
     (effects (font (size 1.27 1.27)) (justify right bottom))
@@
     (effects (font (size 1.27 1.27)) (justify left bottom))
   )
-  (label "STATUS_KTD" (at 81.28 109.22 0)
-    (effects (font (size 1.27 1.27)) (justify left bottom))
-  )
   (label "PD_SDA" (at 314.96 68.58 0)
     (effects (font (size 1.27 1.27)) (justify left bottom))
@@
     (effects (font (size 1.27 1.27)) (justify left bottom))
   )
-  (label "DIAG1" (at 306.07 76.2 180)
-    (effects (font (size 1.27 1.27)) (justify right bottom))
+  (label "DIAG1" (at 233.68 76.2 0)
+    (effects (font (size 1.27 1.27)) (justify left bottom))
   )
   (label "BLUE" (at 81.28 111.76 0)
@@
     (effects (font (size 1.27 1.27)) (justify left bottom))
   )
+  (label "SWO" (at 276.86 111.76 90)
+    (effects (font (size 1.27 1.27)) (justify left bottom))
+  )
   (label "EN2" (at 307.34 203.2 0)
     (effects (font (size 1.27 1.27)) (justify left bottom))
@@
     (effects (font (size 1.27 1.27)) (justify right bottom))
   )
-  (label "DIAG2" (at 306.07 73.66 180)
-    (effects (font (size 1.27 1.27)) (justify right bottom))
+  (label "DIAG2" (at 261.62 111.76 90)
+    (effects (font (size 1.27 1.27)) (justify left bottom))
   )
   (label "SDA_KTD" (at 303.53 68.58 0)
