File: latest/Viewer/main-board.kicad_sch (KiCad schematic)
At the start: 66 parts, among them J1 USB_C_Receptacle_USB2.0_16P, J2 S4B-XH-A_LF__SN_, J3 S4B-XH-A_LF__SN_, J4 Conn_ARM_JTAG_SWD_10, Q1 AONR21307, U1 HUSB238_xxxDD, U2 AP63205WU, U3 AP2112K-3.3, U4 PTR54L, U5 TMC2226-SA, U6 TMC2226-SA, U7 KTD2026BEWE-TR

Commit message: Update latest build (main@ef95290)
Connections:
- no-connect marks 16 -> 29
Changed lines of the file:
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@@
   (junction (at 232.41 180.34) (diameter 0) (color 0 0 0 0)
   )
+  (no_connect (at 243.84 63.5))
   (no_connect (at 92.71 109.22))
+  (no_connect (at 287.02 88.9))
   (no_connect (at 243.84 78.74))
   (no_connect (at 355.6 57.15))
   (no_connect (at 198.12 223.52))
+  (no_connect (at 243.84 71.12))
+  (no_connect (at 243.84 66.04))
+  (no_connect (at 274.32 101.6))
+  (no_connect (at 269.24 101.6))
+  (no_connect (at 243.84 68.58))
   (no_connect (at 316.23 213.36))
   (no_connect (at 198.12 213.36))
+  (no_connect (at 271.78 101.6))
   (no_connect (at 243.84 83.82))
+  (no_connect (at 287.02 73.66))
   (no_connect (at 55.88 80.01))
   (no_connect (at 198.12 205.74))
   (no_connect (at 334.01 231.14))
   (no_connect (at 243.84 86.36))
+  (no_connect (at 243.84 73.66))
+  (no_connect (at 287.02 78.74))
   (no_connect (at 215.9 231.14))
   (no_connect (at 316.23 223.52))
   (no_connect (at 316.23 205.74))
   (no_connect (at 55.88 82.55))
+  (no_connect (at 287.02 81.28))
+  (no_connect (at 287.02 71.12))
   (no_connect (at 243.84 81.28))
   (wire (pts (xy 189.23 172.72) (xy 189.23 170.18))

Commit message: Update latest build (main@23982f9)
Connections:
- net BUTTON: no longer S1.2
- net GND: now also S1.2
Changed lines of the file:
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@@
   (junction (at 110.49 44.45) (diameter 0) (color 0 0 0 0)
-  )
-  (junction (at 356.87 107.95) (diameter 0) (color 0 0 0 0)
   )
   (junction (at 96.52 80.01) (diameter 0) (color 0 0 0 0)
@@
     (stroke (width 0) (type default))
   )
-  (wire (pts (xy 356.87 107.95) (xy 356.87 109.22))
-    (stroke (width 0) (type default))
-  )
   (wire (pts (xy 215.9 160.02) (xy 218.44 160.02))
     (stroke (width 0) (type default))
@@
     (stroke (width 0) (type default))
   )
-  (wire (pts (xy 346.71 107.95) (xy 356.87 107.95))
-    (stroke (width 0) (type default))
-  )
   (wire (pts (xy 346.71 182.88) (xy 368.3 182.88))
     (stroke (width 0) (type default))
@@
     (stroke (width 0) (type default))
   )
+  (wire (pts (xy 354.33 109.22) (xy 356.87 109.22))
+    (stroke (width 0) (type default))
+  )
   (wire (pts (xy 60.96 152.4) (xy 68.58 152.4))
     (stroke (width 0) (type default))
@@
     (stroke (width 0) (type default))
   )
-  (wire (pts (xy 356.87 106.68) (xy 356.87 107.95))
-    (stroke (width 0) (type default))
-  )
   (wire (pts (xy 287.02 68.58) (xy 314.96 68.58))
     (stroke (width 0) (type default))
@@
   )
   (wire (pts (xy 140.97 162.56) (xy 140.97 163.83))
+    (stroke (width 0) (type default))
+  )
+  (wire (pts (xy 346.71 106.68) (xy 356.87 106.68))
     (stroke (width 0) (type default))
   )
@@
     (effects (font (size 1.27 1.27)) (justify right bottom))
   )
-  (label "BUTTON" (at 346.71 107.95 0)
+  (label "BUTTON" (at 346.71 106.68 0)
     (effects (font (size 1.27 1.27)) (justify left bottom))
   )
@@
         )
       )
+    )
+  )
+  (symbol (lib_id "power:GND") (at 354.33 109.22 270) (unit 1) (body_style 1)
+    (exclude_from_sim no) (in_bom yes) (on_board yes) (in_pos_files yes) (dnp no) (fields_autoplaced)
+    (property "Reference" "#PWR057" (at 347.98 109.22 0) (do_not_autoplace no) (show_name no) (hide yes)
+      (effects (font (size 1.27 1.27)))
+    )
+    (property "Value" "GND" (at 350.52 109.2199 90) (do_not_autoplace no) (show_name no)
+      (effects (font (size 1.27 1.27)) (justify right))
+    )
+    (property "Footprint" "" (at 354.33 109.22 0) (do_not_autoplace no) (show_name no) (hide yes)
+      (effects (font (size 1.27 1.27)))
+    )
+    (property "Datasheet" "" (at 354.33 109.22 0) (do_not_autoplace no) (show_name no) (hide yes)
+      (effects (font (size 1.27 1.27)))
+    )
+    (property "Description" "Power symbol creates a global label with name \"GND\" , ground" (at 354.33 109.22 0) (do_not_autoplace no) (show_name no) (hide yes)
+      (effects (font (size 1.27 1.27)))
+    )
+    (pin "1")
+    (instances
+      (project "main-board"
+        (path "/fe215afa-a228-4dbb-8560-a0753323a3f2"
+          (reference "#PWR057") (unit 1)
+        )
+      )

Commit message: Update latest build (main@b699deb)
Connections:
- net +3.3V: no longer C36.1, LED1.1, U7.5 (VIN)
- net +5V: now also C36.1, LED1.1, U7.5 (VIN)
Changed lines of the file:
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@@
   (junction (at 233.68 41.91) (diameter 0) (color 0 0 0 0)
   )
-  (junction (at 133.35 119.38) (diameter 0) (color 0 0 0 0)
-  )
   (junction (at 135.89 44.45) (diameter 0) (color 0 0 0 0)
   )
@@
   (junction (at 250.19 182.88) (diameter 0) (color 0 0 0 0)
   )
+  (junction (at 133.35 119.38) (diameter 0) (color 0 0 0 0)
+  )
   (junction (at 50.8 160.02) (diameter 0) (color 0 0 0 0)
   )
@@
     )
   )
+  (symbol (lib_id "power:+5V") (at 133.35 119.38 270) (unit 1) (body_style 1)
+    (exclude_from_sim no) (in_bom yes) (on_board yes) (in_pos_files yes) (dnp no) (fields_autoplaced)
+    (property "Reference" "#PWR051" (at 129.54 119.38 0) (do_not_autoplace no) (show_name no) (hide yes)
+      (effects (font (size 1.27 1.27)))
+    )
+    (property "Value" "+5V" (at 137.16 119.3799 90) (do_not_autoplace no) (show_name no)
+      (effects (font (size 1.27 1.27)) (justify left))
+    )
+    (property "Footprint" "" (at 133.35 119.38 0) (do_not_autoplace no) (show_name no) (hide yes)
+      (effects (font (size 1.27 1.27)))
+    )
+    (property "Datasheet" "" (at 133.35 119.38 0) (do_not_autoplace no) (show_name no) (hide yes)
+      (effects (font (size 1.27 1.27)))
+    )
+    (property "Description" "Power symbol creates a global label with name \"+5V\"" (at 133.35 119.38 0) (do_not_autoplace no) (show_name no) (hide yes)
+      (effects (font (size 1.27 1.27)))
+    )
+    (pin "1")
+    (instances
+      (project "main-board"
+        (path "/fe215afa-a228-4dbb-8560-a0753323a3f2"
+          (reference "#PWR051") (unit 1)
+        )
+      )
+    )
+  )
   (symbol (lib_id "power:GND") (at 350.52 166.37 180) (unit 1) (body_style 1)
     (exclude_from_sim no) (in_bom yes) (on_board yes) (in_pos_files yes) (dnp no) (fields_autoplaced)
@@
     )
   )
+  (symbol (lib_id "power:+5V") (at 186.69 124.46 270) (unit 1) (body_style 1)
+    (exclude_from_sim no) (in_bom yes) (on_board yes) (in_pos_files yes) (dnp no) (fields_autoplaced)
+    (property "Reference" "#PWR052" (at 182.88 124.46 0) (do_not_autoplace no) (show_name no) (hide yes)
+      (effects (font (size 1.27 1.27)))
+    )
+    (property "Value" "+5V" (at 190.5 124.4599 90) (do_not_autoplace no) (show_name no)
+      (effects (font (size 1.27 1.27)) (justify left))
+    )
+    (property "Footprint" "" (at 186.69 124.46 0) (do_not_autoplace no) (show_name no) (hide yes)
+      (effects (font (size 1.27 1.27)))
+    )
+    (property "Datasheet" "" (at 186.69 124.46 0) (do_not_autoplace no) (show_name no) (hide yes)
+      (effects (font (size 1.27 1.27)))
+    )
+    (property "Description" "Power symbol creates a global label with name \"+5V\"" (at 186.69 124.46 0) (do_not_autoplace no) (show_name no) (hide yes)
+      (effects (font (size 1.27 1.27)))
+    )
+    (pin "1")
+    (instances
+      (project "main-board"
+        (path "/fe215afa-a228-4dbb-8560-a0753323a3f2"
+          (reference "#PWR052") (unit 1)
+        )
+      )
+    )
+  )
   (symbol (lib_id "power:+3.3V") (at 226.06 41.91 90) (unit 1) (body_style 1)
     (exclude_from_sim no) (in_bom yes) (on_board yes) (in_pos_files yes) (dnp no) (fields_autoplaced)
@@
     )
   )
-  (symbol (lib_id "power:+3.3V") (at 133.35 119.38 270) (unit 1) (body_style 1)
-    (exclude_from_sim no) (in_bom yes) (on_board yes) (in_pos_files yes) (dnp no) (fields_autoplaced)
-    (property "Reference" "#PWR052" (at 129.54 119.38 0) (do_not_autoplace no) (show_name no) (hide yes)
-      (effects (font (size 1.27 1.27)))
-    )
-    (property "Value" "+3.3V" (at 137.16 119.3799 90) (do_not_autoplace no) (show_name no)
-      (effects (font (size 1.27 1.27)) (justify left))
-    )
-    (property "Footprint" "" (at 133.35 119.38 0) (do_not_autoplace no) (show_name no) (hide yes)
-      (effects (font (size 1.27 1.27)))
-    )
-    (property "Datasheet" "" (at 133.35 119.38 0) (do_not_autoplace no) (show_name no) (hide yes)
-      (effects (font (size 1.27 1.27)))
-    )
-    (property "Description" "Power symbol creates a global label with name \"+3.3V\"" (at 133.35 119.38 0) (do_not_autoplace no) (show_name no) (hide yes)
-      (effects (font (size 1.27 1.27)))
-    )
-    (pin "1")
-    (instances
-      (project "main-board"
-        (path "/fe215afa-a228-4dbb-8560-a0753323a3f2"
-          (reference "#PWR052") (unit 1)
-        )
-      )
-    )
-  )
   (symbol (lib_id "power:GND") (at 172.72 198.12 270) (unit 1) (body_style 1)
     (exclude_from_sim no) (in_bom yes) (on_board yes) (in_pos_files yes) (dnp no) (fields_autoplaced)
@@
         )
       )
-    )
-  )
-  (symbol (lib_id "power:+3.3V") (at 186.69 124.46 270) (unit 1) (body_style 1)
-    (exclude_from_sim no) (in_bom yes) (on_board yes) (in_pos_files yes) (dnp no) (fields_autoplaced)
-    (property "Reference" "#PWR051" (at 182.88 124.46 0) (do_not_autoplace no) (show_name no) (hide yes)
-      (effects (font (size 1.27 1.27)))
-    )
-    (property "Value" "+3.3V" (at 190.5 124.4599 90) (do_not_autoplace no) (show_name no)
-      (effects (font (size 1.27 1.27)) (justify left))
-    )
-    (property "Footprint" "" (at 186.69 124.46 0) (do_not_autoplace no) (show_name no) (hide yes)
-      (effects (font (size 1.27 1.27)))
-    )
-    (property "Datasheet" "" (at 186.69 124.46 0) (do_not_autoplace no) (show_name no) (hide yes)
-      (effects (font (size 1.27 1.27)))
-    )
-    (property "Description" "Power symbol creates a global label with name \"+3.3V\"" (at 186.69 124.46 0) (do_not_autoplace no) (show_name no) (hide yes)
-      (effects (font (size 1.27 1.27)))
-    )
-    (pin "1")
-    (instances
-      (project "main-board"
-        (path "/fe215afa-a228-4dbb-8560-a0753323a3f2"
-          (reference "#PWR051") (unit 1)
-        )
-      )

Commit message: Update latest build (main@6be02d9)
Parts:
- added D1: SMBJ16A, DIOM5436X261N, symbol Samacsys:SMBJ16A
- added D2: SS34, Diode_SMD:D_SMA, symbol Diode:SS34
Connections:
- net GND: now also D1.2 (A)
- net VBUS: now also D1.1 (K), D2.1 (K); no longer Q1.5 (D_1), Q1.6 (D_2), Q1.7 (D_3), Q1.8 (D_4)
- new net: D2.2 (A), Q1.5 (D_1), Q1.6 (D_2), Q1.7 (D_3), Q1.8 (D_4)
Changed lines of the file:
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@@
     (stroke (width 0) (type default))
   )
-  (wire (pts (xy 135.89 36.83) (xy 143.51 36.83))
-    (stroke (width 0) (type default))
-  )
   (wire (pts (xy 193.04 149.86) (xy 193.04 157.48))
     (stroke (width 0) (type default))
@@
     )
   )
+  (symbol (lib_id "Diode:SS34") (at 139.7 36.83 180) (unit 1) (body_style 1)
+    (exclude_from_sim no) (in_bom yes) (on_board yes) (in_pos_files yes) (dnp no) (fields_autoplaced)
+    (property "Reference" "D2" (at 140.0175 30.48 0) (do_not_autoplace no) (show_name no)
+      (effects (font (size 1.27 1.27)))
+    )
+    (property "Value" "SS34" (at 140.0175 33.02 0) (do_not_autoplace no) (show_name no)
+      (effects (font (size 1.27 1.27)))
+    )
+    (property "Footprint" "Diode_SMD:D_SMA" (at 139.7 32.385 0) (do_not_autoplace no) (show_name no) (hide yes)
+      (effects (font (size 1.27 1.27)))
+    )
+    (property "Datasheet" "https://www.vishay.com/docs/88751/ss32.pdf" (at 139.7 36.83 0) (do_not_autoplace no) (show_name no) (hide yes)
+      (effects (font (size 1.27 1.27)))
+    )
+    (property "Description" "40V 3A Schottky Diode, SMA" (at 139.7 36.83 0) (do_not_autoplace no) (show_name no) (hide yes)
+      (effects (font (size 1.27 1.27)))
+    )
+    (pin "2")
+    (pin "1")
+    (instances
+      (project "main-board"
+        (path "/fe215afa-a228-4dbb-8560-a0753323a3f2"
+          (reference "D2") (unit 1)
+        )
+      )
+    )
+  )
   (symbol (lib_id "Device:R") (at 99.06 52.07 90) (unit 1) (body_style 1)
     (exclude_from_sim no) (in_bom yes) (on_board yes) (in_pos_files yes) (dnp no)
@@
     )
   )
+  (symbol (lib_id "power:VBUS") (at 190.5 36.83 0) (unit 1) (body_style 1)
+    (exclude_from_sim no) (in_bom yes) (on_board yes) (in_pos_files yes) (dnp no) (fields_autoplaced)
+    (property "Reference" "#PWR059" (at 190.5 40.64 0) (do_not_autoplace no) (show_name no) (hide yes)
+      (effects (font (size 1.27 1.27)))
+    )
+    (property "Value" "VBUS" (at 190.5 31.75 0) (do_not_autoplace no) (show_name no)
+      (effects (font (size 1.27 1.27)))
+    )
+    (property "Footprint" "" (at 190.5 36.83 0) (do_not_autoplace no) (show_name no) (hide yes)
+      (effects (font (size 1.27 1.27)))
+    )
+    (property "Datasheet" "" (at 190.5 36.83 0) (do_not_autoplace no) (show_name no) (hide yes)
+      (effects (font (size 1.27 1.27)))
+    )
+    (property "Description" "Power symbol creates a global label with name \"VBUS\"" (at 190.5 36.83 0) (do_not_autoplace no) (show_name no) (hide yes)
+      (effects (font (size 1.27 1.27)))
+    )
+    (pin "1")
+    (instances
+      (project "main-board"
+        (path "/fe215afa-a228-4dbb-8560-a0753323a3f2"
+          (reference "#PWR059") (unit 1)
+        )
+      )
+    )
+  )
   (symbol (lib_id "Device:C") (at 171.45 173.99 180) (unit 1) (body_style 1)
     (exclude_from_sim no) (in_bom yes) (on_board yes) (in_pos_files yes) (dnp no) (fields_autoplaced)
@@
     )
   )
+  (symbol (lib_id "power:GND") (at 190.5 52.07 0) (unit 1) (body_style 1)
+    (exclude_from_sim no) (in_bom yes) (on_board yes) (in_pos_files yes) (dnp no) (fields_autoplaced)
+    (property "Reference" "#PWR058" (at 190.5 58.42 0) (do_not_autoplace no) (show_name no) (hide yes)
+      (effects (font (size 1.27 1.27)))
+    )
+    (property "Value" "GND" (at 190.5 57.15 0) (do_not_autoplace no) (show_name no)
+      (effects (font (size 1.27 1.27)))
+    )
+    (property "Footprint" "" (at 190.5 52.07 0) (do_not_autoplace no) (show_name no) (hide yes)
+      (effects (font (size 1.27 1.27)))
+    )
+    (property "Datasheet" "" (at 190.5 52.07 0) (do_not_autoplace no) (show_name no) (hide yes)
+      (effects (font (size 1.27 1.27)))
+    )
+    (property "Description" "Power symbol creates a global label with name \"GND\" , ground" (at 190.5 52.07 0) (do_not_autoplace no) (show_name no) (hide yes)
+      (effects (font (size 1.27 1.27)))
+    )
+    (pin "1")
+    (instances
+      (project "main-board"
+        (path "/fe215afa-a228-4dbb-8560-a0753323a3f2"
+          (reference "#PWR058") (unit 1)
+        )
+      )
+    )
+  )
   (symbol (lib_id "Device:R") (at 176.53 195.58 270) (unit 1) (body_style 1)
     (exclude_from_sim no) (in_bom yes) (on_board yes) (in_pos_files yes) (dnp no)
@@
         )
       )
+    )
+  )
+  (symbol (lib_id "Samacsys:SMBJ16A") (at 190.5 36.83 270) (unit 1) (body_style 1)
+    (exclude_from_sim no) (in_bom yes) (on_board yes) (in_pos_files yes) (dnp no) (fields_autoplaced)
+    (property "Reference" "D1" (at 194.31 42.6719 90) (do_not_autoplace no) (show_name no)
+      (effects (font (size 1.27 1.27)) (justify left))
+    )
+    (property "Value" "SMBJ16A" (at 194.31 45.2119 90) (do_not_autoplace no) (show_name no)
+      (effects (font (size 1.27 1.27)) (justify left))
+    )
+    (property "Footprint" "DIOM5436X261N" (at 96.85 46.99 0) (do_not_autoplace no) (show_name no) (hide yes)
+      (effects (font (size 1.27 1.27)) (justify left bottom))
+    )
+    (property "Datasheet" "https://datasheet.datasheetarchive.com/originals/dk/DKDS-14/271386.pdf" (at -3.15 46.99 0) (do_not_autoplace no) (show_name no) (hide yes)
+      (effects (font (size 1.27 1.27)) (justify left bottom))
+    )
+    (property "Description" "TVS Diode Single Uni-Dir 16V 600W 2-Pin SMB T/R" (at 190.5 36.83 0) (do_not_autoplace no) (show_name no) (hide yes)
+      (effects (font (size 1.27 1.27)))
+    )
+    (property "Height" "2.61" (at -203.15 46.99 0) (do_not_autoplace no) (show_name no) (hide yes)
+      (effects (font (size 1.27 1.27)) (justify left bottom))
+    )
+    (property "Manufacturer_Name" "LITTELFUSE" (at -303.15 46.99 0) (do_not_autoplace no) (show_name no) (hide yes)
+      (effects (font (size 1.27 1.27)) (justify left bottom))
+    )
+    (property "Manufacturer_Part_Number" "SMBJ16A" (at -403.15 46.99 0) (do_not_autoplace no) (show_name no) (hide yes)
+      (effects (font (size 1.27 1.27)) (justify left bottom))
+    )
+    (property "Mouser Part Number" "576-SMBJ16A" (at -503.15 46.99 0) (do_not_autoplace no) (show_name no) (hide yes)
+      (effects (font (size 1.27 1.27)) (justify left bottom))
+    )
+    (property "Mouser Price/Stock" "https://www.mouser.co.uk/ProductDetail/Littelfuse/SMBJ16A?qs=HR2RnyOI4E4LWSQFq1tisQ%3D%3D" (at -603.15 46.99 0) (do_not_autoplace no) (show_name no) (hide yes)
+      (effects (font (size 1.27 1.27)) (justify left bottom))
+    )
+    (property "Arrow Part Number" "SMBJ16A" (at -703.15 46.99 0) (do_not_autoplace no) (show_name no) (hide yes)
+      (effects (font (size 1.27 1.27)) (justify left bottom))
+    )
+    (property "Arrow Price/Stock" "https://www.arrow.com/en/products/smbj16a/littelfuse?utm_currency=USD&region=nac" (at -803.15 46.99 0) (do_not_autoplace no) (show_name no) (hide yes)
+      (effects (font (size 1.27 1.27)) (justify left bottom))
+    )
+    (pin "1")
+    (pin "2")
+    (instances
+      (project "main-board"
+        (path "/fe215afa-a228-4dbb-8560-a0753323a3f2"
+          (reference "D1") (unit 1)
+        )
+      )

Commit message: Update latest build (main@5ff42ea)
Parts:
- R4: value 10R -> 14K; now fitted
- R5: value 10R -> 16K5
Changed lines of the file:
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@@
       (effects (font (size 1.27 1.27)) (justify right))
     )
-    (property "Value" "10R" (at 93.98 76.1999 0) (do_not_autoplace no) (show_name no)
+    (property "Value" "16K5" (at 93.98 76.1999 0) (do_not_autoplace no) (show_name no)
       (effects (font (size 1.27 1.27)) (justify right))
     )
@@
   )
   (symbol (lib_id "Device:R") (at 101.6 74.93 0) (unit 1) (body_style 1)
-    (exclude_from_sim no) (in_bom yes) (on_board yes) (in_pos_files no) (dnp yes) (fields_autoplaced)
+    (exclude_from_sim no) (in_bom yes) (on_board yes) (in_pos_files yes) (dnp no) (fields_autoplaced)
     (property "Reference" "R4" (at 104.14 73.6599 0) (do_not_autoplace no) (show_name no)
       (effects (font (size 1.27 1.27)) (justify left))
     )
-    (property "Value" "10R" (at 104.14 76.1999 0) (do_not_autoplace no) (show_name no)
-      (effects (font (size 1.27 1.27)) (justify left))
-    )
+    (property "Value" "14K" (at 104.14 76.1999 0) (do_not_autoplace no) (show_name no)
+      (effects (font (size 1.27 1.27)) (justify left))
+    )

Commit message: Update latest build (main@4fe8fca)
Parts:
- R5: now fitted
Changed lines of the file:
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@@
   )
   (symbol (lib_id "Device:R") (at 91.44 74.93 180) (unit 1) (body_style 1)
-    (exclude_from_sim no) (in_bom yes) (on_board yes) (in_pos_files no) (dnp yes) (fields_autoplaced)
+    (exclude_from_sim no) (in_bom yes) (on_board yes) (in_pos_files yes) (dnp no) (fields_autoplaced)
     (property "Reference" "R5" (at 93.98 73.6599 0) (do_not_autoplace no) (show_name no)
       (effects (font (size 1.27 1.27)) (justify right))
