File: latest/Viewer/main-board.kicad_sch (KiCad schematic)
At the start: 68 parts, among them J1 USB_C_Receptacle_USB2.0_16P, J2 S4B-XH-A_LF__SN_, J3 S4B-XH-A_LF__SN_, J4 Conn_ARM_JTAG_SWD_10, Q1 AONR21307, U1 HUSB238_xxxDD, U2 AP63205WU, U3 AP2112K-3.3, U4 PTR54L, U5 TMC2226-SA, U6 TMC2226-SA, U7 KTD2026BEWE-TR

Commit message: Update latest build (main@5c34972)
Other:
- moved on the sheet: C20
Changed lines of the file:
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@@
     (stroke (width 0) (type default))
   )
-  (wire (pts (xy 245.11 160.02) (xy 257.81 160.02))
-    (stroke (width 0) (type default))
-  )
   (wire (pts (xy 81.28 234.95) (xy 77.47 234.95))
     (stroke (width 0) (type default))
@@
     (stroke (width 0) (type default))
   )
-  (wire (pts (xy 245.11 147.32) (xy 257.81 147.32))
-    (stroke (width 0) (type default))
-  )
   (wire (pts (xy 266.7 101.6) (xy 266.7 111.76))
     (stroke (width 0) (type default))
@@
   (netclass_flag "" (length 2.54) (shape round) (at 401.32 138.43 0)
     (effects (font (size 1.27 1.27)) (justify left bottom))
-    (property "Netclass" "Default" (at 402.0185 135.89 0) (do_not_autoplace no) (show_name no) (hide yes)
+    (property "Netclass" "DRV2" (at 402.0185 135.89 0) (do_not_autoplace no) (show_name no) (hide yes)
       (effects (font (size 1.27 1.27)) (justify left))
     )
@@
   (netclass_flag "" (length 2.54) (shape round) (at 278.13 138.43 0)
     (effects (font (size 1.27 1.27)) (justify left bottom))
-    (property "Netclass" "Default" (at 278.8285 135.89 0) (do_not_autoplace no) (show_name no) (hide yes)
+    (property "Netclass" "DRV1" (at 278.8285 135.89 0) (do_not_autoplace no) (show_name no) (hide yes)
       (effects (font (size 1.27 1.27)) (justify left))
     )
-    (property "Component Class" "DRV1" (at 278.13 133.858 0) (do_not_autoplace no) (show_name no)
+    (property "Component Class" "DRV1" (at 278.892 133.858 0) (do_not_autoplace no) (show_name no)
       (effects (font (size 1.27 1.27) (italic yes)) (justify left))
     )
@@
     )
   )
-  (symbol (lib_id "Samacsys:EEE-FT1V101AP") (at 257.81 160.02 90) (unit 1) (body_style 1)
+  (symbol (lib_id "power:GND") (at 218.44 106.68 180) (unit 1) (body_style 1)
+    (exclude_from_sim no) (in_bom yes) (on_board yes) (in_pos_files yes) (dnp no) (fields_autoplaced)
+    (property "Reference" "#PWR061" (at 218.44 100.33 0) (do_not_autoplace no) (show_name no) (hide yes)
+      (effects (font (size 1.27 1.27)))
+    )
+    (property "Value" "GND" (at 218.44 101.6 0) (do_not_autoplace no) (show_name no)
+      (effects (font (size 1.27 1.27)))
+    )
+    (property "Footprint" "" (at 218.44 106.68 0) (do_not_autoplace no) (show_name no) (hide yes)
+      (effects (font (size 1.27 1.27)))
+    )
+    (property "Datasheet" "" (at 218.44 106.68 0) (do_not_autoplace no) (show_name no) (hide yes)
+      (effects (font (size 1.27 1.27)))
+    )
+    (property "Description" "Power symbol creates a global label with name \"GND\" , ground" (at 218.44 106.68 0) (do_not_autoplace no) (show_name no) (hide yes)
+      (effects (font (size 1.27 1.27)))
+    )
+    (pin "1")
+    (instances
+      (project "main-board"
+        (path "/fe215afa-a228-4dbb-8560-a0753323a3f2"
+          (reference "#PWR061") (unit 1)
+        )
+      )
+    )
+  )
+  (symbol (lib_id "Samacsys:EEE-FT1V101AP") (at 218.44 119.38 90) (unit 1) (body_style 1)
     (exclude_from_sim no) (in_bom yes) (on_board yes) (in_pos_files yes) (dnp no) (fields_autoplaced)
-    (property "Reference" "C20" (at 261.62 152.3999 90) (do_not_autoplace no) (show_name no)
+    (property "Reference" "C20" (at 222.25 111.7599 90) (do_not_autoplace no) (show_name no)
       (effects (font (size 1.27 1.27)) (justify right))
     )
-    (property "Value" "EEE-FT1V101AP" (at 261.62 154.9399 90) (do_not_autoplace no) (show_name no)
+    (property "Value" "EEE-FT1V101AP" (at 222.25 114.2999 90) (do_not_autoplace no) (show_name no)
       (effects (font (size 1.27 1.27)) (justify right))
     )
-    (property "Footprint" "EEE1AA101SP" (at 354 151.13 0) (do_not_autoplace no) (show_name no) (hide yes)
+    (property "Footprint" "EEE1AA101SP" (at 314.63 110.49 0) (do_not_autoplace no) (show_name no) (hide yes)
       (effects (font (size 1.27 1.27)) (justify left top))
     )
-    (property "Datasheet" "http://industrial.panasonic.com/cdbs/www-data/pdf/RDE0000/ABA0000C1240.pdf" (at 454 151.13 0) (do_not_autoplace no) (show_name no) (hide yes)
+    (property "Datasheet" "http://industrial.panasonic.com/cdbs/www-data/pdf/RDE0000/ABA0000C1240.pdf" (at 414.63 110.49 0) (do_not_autoplace no) (show_name no) (hide yes)
       (effects (font (size 1.27 1.27)) (justify left top))
     )
-    (property "Description" "Aluminum Electrolytic Capacitors - SMD 100uF 35volts 6.3x5.8mm SMD" (at 257.81 160.02 0) (do_not_autoplace no) (show_name no) (hide yes)
+    (property "Description" "Aluminum Electrolytic Capacitors - SMD 100uF 35volts 6.3x5.8mm SMD" (at 218.44 119.38 0) (do_not_autoplace no) (show_name no) (hide yes)
       (effects (font (size 1.27 1.27)))
     )
-    (property "Height" "7.8" (at 654 151.13 0) (do_not_autoplace no) (show_name no) (hide yes)
+    (property "Height" "7.8" (at 614.63 110.49 0) (do_not_autoplace no) (show_name no) (hide yes)
       (effects (font (size 1.27 1.27)) (justify left top))
     )
-    (property "Manufacturer_Name" "Panasonic" (at 754 151.13 0) (do_not_autoplace no) (show_name no) (hide yes)
+    (property "Manufacturer_Name" "Panasonic" (at 714.63 110.49 0) (do_not_autoplace no) (show_name no) (hide yes)
       (effects (font (size 1.27 1.27)) (justify left top))
     )
-    (property "Manufacturer_Part_Number" "EEE-FT1V101AP" (at 854 151.13 0) (do_not_autoplace no) (show_name no) (hide yes)
+    (property "Manufacturer_Part_Number" "EEE-FT1V101AP" (at 814.63 110.49 0) (do_not_autoplace no) (show_name no) (hide yes)
       (effects (font (size 1.27 1.27)) (justify left top))
     )
-    (property "Mouser Part Number" "667-EEE-FT1V101AP" (at 954 151.13 0) (do_not_autoplace no) (show_name no) (hide yes)
+    (property "Mouser Part Number" "667-EEE-FT1V101AP" (at 914.63 110.49 0) (do_not_autoplace no) (show_name no) (hide yes)
       (effects (font (size 1.27 1.27)) (justify left top))
     )
-    (property "Mouser Price/Stock" "https://www.mouser.co.uk/ProductDetail/Panasonic/EEE-FT1V101AP?qs=CMJjuEs1%252BuEsbOqam%2FkTqg%3D%3D" (at 1054 151.13 0) (do_not_autoplace no) (show_name no) (hide yes)
+    (property "Mouser Price/Stock" "https://www.mouser.co.uk/ProductDetail/Panasonic/EEE-FT1V101AP?qs=CMJjuEs1%252BuEsbOqam%2FkTqg%3D%3D" (at 1014.63 110.49 0) (do_not_autoplace no) (show_name no) (hide yes)
       (effects (font (size 1.27 1.27)) (justify left top))
     )
-    (property "Arrow Part Number" "EEE-FT1V101AP" (at 1154 151.13 0) (do_not_autoplace no) (show_name no) (hide yes)
+    (property "Arrow Part Number" "EEE-FT1V101AP" (at 1114.63 110.49 0) (do_not_autoplace no) (show_name no) (hide yes)
       (effects (font (size 1.27 1.27)) (justify left top))
     )
-    (property "Arrow Price/Stock" "https://www.arrow.com/en/products/eeeft1v101ap/panasonic.html?utm_currency=USD&region=nac" (at 1254 151.13 0) (do_not_autoplace no) (show_name no) (hide yes)
+    (property "Arrow Price/Stock" "https://www.arrow.com/en/products/eeeft1v101ap/panasonic.html?utm_currency=USD&region=nac" (at 1214.63 110.49 0) (do_not_autoplace no) (show_name no) (hide yes)
       (effects (font (size 1.27 1.27)) (justify left top))
     )
@@
         )
       )
+    )
+  )
+  (symbol (lib_id "power:VBUS") (at 218.44 119.38 180) (unit 1) (body_style 1)
+    (exclude_from_sim no) (in_bom yes) (on_board yes) (in_pos_files yes) (dnp no) (fields_autoplaced)
+    (property "Reference" "#PWR060" (at 218.44 115.57 0) (do_not_autoplace no) (show_name no) (hide yes)
+      (effects (font (size 1.27 1.27)))
+    )
+    (property "Value" "VBUS" (at 218.44 124.46 0) (do_not_autoplace no) (show_name no)
+      (effects (font (size 1.27 1.27)))
+    )
+    (property "Footprint" "" (at 218.44 119.38 0) (do_not_autoplace no) (show_name no) (hide yes)
+      (effects (font (size 1.27 1.27)))
+    )
+    (property "Datasheet" "" (at 218.44 119.38 0) (do_not_autoplace no) (show_name no) (hide yes)
+      (effects (font (size 1.27 1.27)))
+    )
+    (property "Description" "Power symbol creates a global label with name \"VBUS\"" (at 218.44 119.38 0) (do_not_autoplace no) (show_name no) (hide yes)
+      (effects (font (size 1.27 1.27)))
+    )
+    (pin "1")
+    (instances
+      (project "main-board"
+        (path "/fe215afa-a228-4dbb-8560-a0753323a3f2"
+          (reference "#PWR060") (unit 1)
+        )
+      )
